File: schematics/oven_high_voltage.sch (EAGLE design)
At the start: 6 parts, among them M1 Convection Fan

Commit message: Update earth and chassis ground symbols.
Connections:
- net 3.3V renamed GND
Changed lines of the file:
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@@
 <part name="P1" library="con-lstb" library_urn="urn:adsk.eagle:library:162" deviceset="MA05-1" device="" package3d_urn="urn:adsk.eagle:package:8332/1"/>
 <part name="M1" library="SparkFun-Electromechanical" deviceset="MOTOR" device="10MM" value="Convection Fan"/>
-<part name="GND1" library="SparkFun-PowerSymbols" deviceset="GND2" device="" value="Chassis Ground"/>
 <part name="FRAME1" library="frames" deviceset="LETTER_L" device="">
 <attribute name="COMPANY_NAME" value="An Alex McLain Design"/>
@@
 <attribute name="TITLE" value="OVEN HIGH VOLTAGE"/>
 </part>
+<part name="GND1" library="supply" deviceset="CGND" device=""/>
 </parts>
 <sheets>
@@
 <attribute name="VALUE" x="130.81" y="88.646" size="1.778" layer="96" font="vector"/>
 </instance>
-<instance part="GND1" gate="G$1" x="104.14" y="81.28" smashed="yes">
-<attribute name="VALUE" x="104.14" y="77.724" size="1.778" layer="96" align="top-center"/>
-</instance>
 <instance part="FRAME1" gate="G$1" x="0" y="0">
 <attribute name="COMPANY_NAME" x="0" y="0" size="1.778" layer="96" display="off"/>
@@
 </instance>
 <instance part="FRAME1" gate="G$2" x="147.32" y="0"/>
+<instance part="GND1" gate="1" x="104.14" y="81.28"/>
 </instances>
 <busses>
@@
 </segment>
 </net>
-<net name="3.3V" class="0">
+<net name="GND" class="0">
 <segment>
 <pinref part="P1" gate="G$1" pin="5"/>
-<pinref part="GND1" gate="G$1" pin="3.3V"/>
 <wire x1="101.6" y1="88.9" x2="104.14" y2="88.9" width="0.1524" layer="91"/>
 <wire x1="104.14" y1="88.9" x2="104.14" y2="83.82" width="0.1524" layer="91"/>
+<pinref part="GND1" gate="1" pin="GND"/>
 </segment>
 </net>
